File: hardware/PC_and_Light_Controller.kicad_pcb (KiCad board)
At the start: 2 copper layers, 81.2 x 58.9 mm, 30 parts, among them J1 Screw_Terminal_01x04, J3 Screw_Terminal_01x06, J4 Screw_Terminal_01x06, U1 ESP32-DEVKIT-V1, U2 TPS259807ONRGER, U3 TPS259807ONRGER, U4 TPS259807ONRGER

Commit message: Manufacturing Readiness
Routing:
- net GND: vias 6 -> 7
- added copper zone on B.Cu, net GND
Other:
- board text added: "https://github.com/HighCarlSagan/PC_and_Light_Controller"
Changed lines of the file:
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@@
 		)
 	)
+	(gr_text "https://github.com/HighCarlSagan/PC_and_Light_Controller"
+		(at 90.24 28.63 0)
+		(layer "B.SilkS")
+		(effects
+			(font
+				(size 1 1)
+				(thickness 0.1)
+			)
+			(justify left bottom mirror)
+		)
+	)
 	(segment
 		(start 83.6942 32.8975)
@@
 	)
 	(via
+		(at 43.19 29.43)
+		(size 0.6)
+		(drill 0.3)
+		(layers "F.Cu" "B.Cu")
+		(free yes)
+		(net 2)
+	)
+	(via
 		(at 54.225 39.6575)
 		(size 0.6)
@@
 			)
 		)
+	)
+	(zone
+		(net 2)
+		(net_name "GND")
+		(layers "F.Cu" "B.Cu")
+		(hatch edge 0.5)
+		(priority 2)
+		(connect_pads
+			(clearance 0.5)
+		)
+		(min_thickness 0.25)
+		(filled_areas_thickness no)
+		(fill yes
+			(thermal_gap 0.5)
+			(thermal_bridge_width 0.5)
+		)
+		(polygon
+			(pts
+				(xy 33.08 16.15) (xy 114.31 16.14) (xy 114.31 75.03) (xy 33.08 75.02)
+			)
+		)

Commit message: Final final manufacturing ready board
Parts:
- removed REF**: KiCad-Logo2_5mm_SilkScreen, Symbol:KiCad-Logo2_5mm_SilkScreen
- removed REF**: OSHW-Logo2_7.3x6mm_SilkScreen, Symbol:OSHW-Logo2_7.3x6mm_SilkScreen
- added H1: MountingHole_Pad, MountingHole:MountingHole_2.2mm_M2_Pad_Via, F.Cu at (36.7, 19.7)
- added H2: MountingHole_Pad, MountingHole:MountingHole_2.2mm_M2_Pad_Via, F.Cu at (110.5, 19.7)
- added H3: MountingHole_Pad, MountingHole:MountingHole_2.2mm_M2_Pad_Via, F.Cu at (36.7, 71.5)
- added H4: MountingHole_Pad, MountingHole:MountingHole_2.2mm_M2_Pad_Via, F.Cu at (110.5, 71.5)
- moved R13 13.9 mm to (59.2, 43.3), turned to 180 degrees
- moved J4 13.9 mm to (107.4, 53.2)
- moved C2 13.8 mm to (56.0, 24.2), turned to -90 degrees
- moved J3 5.72 mm to (40.5, 37.9)
- moved C5 4.35 mm to (40.9, 30.7), turned to 0 degrees
Connections:
- U1 pad 10: unconnected-(U1-D19-Pad10) -> /LED_2_CTRL
- U1 pad 15: unconnected-(U1-D23-Pad15) -> /LED_1_CTRL
- U1 pad 23: /LED_1_CTRL -> unconnected-(U1-D25-Pad23)
- U1 pad 24: /LED_2_CTRL -> unconnected-(U1-D26-Pad24)
- U1 pad 25: /LED_3_CTRL -> unconnected-(U1-D27-Pad25)
- U1 pad 4: unconnected-(U1-D2-Pad4) -> /LED_3_CTRL
Routing:
- net +5V: track 290.6 -> 220.8 mm, vias 2 -> 5
- net /LED_2_CTRL: track 74.1 -> 7.45 mm, vias 2 -> 1
- net /LED_1_CTRL: track 60.3 -> 7.92 mm, vias 2 -> 1
- net /LED_3_CTRL: track 58.4 -> 7.72 mm, vias 4 -> 1
- net Net-(U1-TX0): track 15.7 -> 2.61 mm
- net /Motor_PWM: track 8.09 -> 19.9 mm
- net /LED_1_VOUT: track 107.3 -> 95.9 mm, vias 3 -> 1
- net GND: track 454.6 -> 450.5 mm, vias 7 -> 9
- net /LED_2_VOUT: track 75.6 -> 71.6 mm, vias 2 -> 1
- net /LED_3_VOUT: track 49.0 -> 50.6 mm, vias 1 -> 3
- removed copper zone on B.Cu, net GND
Other:
- board text added: "Motor Drive"
- board text added: "UPS_Light_Control"
- board text removed: "PC_and_Lighting_Controller"
